Commit message: initial commit

File: urdf/sick_ldmrs.urdf.xacro (robot description, xacro)
@@ -1,5 +1,5 @@
 <?xml version="1.0"?>
-<robot name="sensor_hokuyo_utm30lx" xmlns:xacro="http://www.ros.org/wiki/xacro">
-  <xacro:macro name="sensor_hokuyo_utm30lx" params="name parent *origin min_angle:=-2.0943 max_angle:=2.0943">
+<robot name="sensor_sick_ldmrs" xmlns:xacro="http://www.ros.org/wiki/xacro">
+  <xacro:macro name="sensor_sick_ldmrs" params="name parent *origin min_angle:=-2.0943 max_angle:=2.0943">
     <joint name="${name}_joint" type="fixed">
       <!-- FRONT MOUNT  -->
@@ -12,8 +12,14 @@
     </joint>
     <link name="${name}_link">
+      <collision>
+        <origin xyz="0 0 -0.05" rpy="0 0 0"/>
+        <geometry>
+          <box size="0.1 0.1 0.08"/>
+        </geometry>
+      </collision>
       <visual>
-        <origin xyz="0 0 0" rpy="0 0 0"/>
+        <origin xyz="0 0 -0.05" rpy="0 0 0"/>
         <geometry>
-            <mesh filename="package://robotnik_sensors/meshes/hokuyo_utm_30lx.dae"/>
+            <mesh filename="package://robotnik_sensors/meshes/hokuyo_urg_04lx.dae"/>
         </geometry>
       </visual>
@@ -25,7 +31,7 @@
     </link>
     <!-- Hokuyo sensor for simulation -->
-    <sensor_hokuyo_utm_gazebo/>
+    <sensor_sick_ldmrs_gazebo/>
   </xacro:macro>
-  <xacro:macro name="sensor_hokuyo_utm_gazebo">
+  <xacro:macro name="sensor_sick_ldmrs_gazebo">
     <gazebo reference="${name}_link">
 			<sensor type="ray" name="${name}_sensor">
@@ -58,5 +64,5 @@
 				</plugin>
 			</sensor>
-		</gazebo>
+	</gazebo>
   </xacro:macro>
 </robot>
